Commit message: fix: fix some simulation issues
Details are as below:
1. Change the camera joints pose in qrb_robot_base_mini URDF
2. Fix odom error of robot base by setting the <mu> value of caster_wheel_link to zero,
removing dynamics tag in qrb_robot_base and mini URDF and friction tag of warehouse.sdf
3. Change the rgbd camera to depth camera and remapping the ROS topic of depth image
4. Remove the intrinsics tags of depth camera
5. Change the default parameters of rgb camera, depth camera,imu and laser
6. Change the default robot namespace of qrb_robot_base_mini
7. Change the default shell to bash in docker_build.sh
8. Move worlds folder from qrb_ros_sim_description to qrb_ros_sim_gazebo

Signed-off-by: weijshen <weijshen@qti.qualcomm.com>

File: qrb_ros_sim_gazebo/urdf/gazebo_qrb_robot_base.urdf.xacro (robot description, xacro)
@@ -25,7 +25,7 @@
   <!-- Gazebo Plugins -->
   <!-- gz-sim-diff-drive-system controller -->
-  <xacro:property name="separation_multiplier" value="1.15"/>
+  <xacro:property name="separation_multiplier" value="1.1525"/>
   <xacro:property name="radius_multiplier" value="1.0"/>
-  <xacro:property name="odom_update_rate" value="30"/>
+  <xacro:property name="odom_update_rate" value="50"/>
   <xacro:include filename="$(find qrb_ros_sim_gazebo)/urdf/xacro/gazebo_qrb_robot_base_diff_drive.xacro" />
   <xacro:qrb_robot_base_diff_drive ns="$(arg robot_base_ns)" wheel_separation="${wheel_separation}" separation_multiplier="${separation_multiplier}"

File: qrb_ros_sim_gazebo/urdf/gazebo_qrb_robot_base_mini.urdf.xacro (robot description, xacro)
@@ -39,7 +39,7 @@
   <!-- Gazebo Plugins -->
   <!-- gz-sim-diff-drive-system controller -->
-  <xacro:property name="separation_multiplier" value="1.15"/>
+  <xacro:property name="separation_multiplier" value="1.125"/>
   <xacro:property name="radius_multiplier" value="1.0"/>
-  <xacro:property name="odom_update_rate" value="30"/>
+  <xacro:property name="odom_update_rate" value="50"/>
   <xacro:include filename="$(find qrb_ros_sim_gazebo)/urdf/xacro/gazebo_qrb_robot_base_diff_drive.xacro" />
   <xacro:qrb_robot_base_diff_drive ns="$(arg robot_base_ns)" wheel_separation="${wheel_separation}" separation_multiplier="${separation_multiplier}"

File: qrb_ros_sim_gazebo/urdf/xacro/gazebo_depth_camera.xacro (robot description, xacro)
@@ -5,23 +5,13 @@
     <xacro:property name="depth_camera_params" value="${xacro.load_yaml(depth_camera_params_yaml_path)}"/>
     <xacro:property name="depth_camera_sub" value="${depth_camera_params['camera']}"/>
-    <xacro:property name="depth_camera_sub_lens_intri" value="${depth_camera_sub['lens']['intrinsics']}"/>
     <xacro:property name="depth_camera_sub_image" value="${depth_camera_sub['image']}"/>
     <xacro:property name="depth_camera_sub_clip" value="${depth_camera_sub['depth_camera']['clip']}"/>
     <xacro:property name="depth_camera_sub_noise" value="${depth_camera_sub['noise']}"/>
     <gazebo reference="${reference_link}">
-    <sensor name="${namespace}${depth_camera_params['sensor_name']}" type="rgbd_camera">
+    <sensor name="${namespace}${depth_camera_params['sensor_name']}" type="depth_camera">
       <update_rate>${depth_camera_params['update_rate']}</update_rate>
       <camera>
         <optical_frame_id>${reference_link}</optical_frame_id>
         <horizontal_fov>${depth_camera_sub['horizontal_fov']}</horizontal_fov>
-        <lens>
-          <intrinsics>
-            <fx>${depth_camera_sub_lens_intri['fx']}</fx>
-            <fy>${depth_camera_sub_lens_intri['fy']}</fy>
-            <cx>${depth_camera_sub_lens_intri['cx']}</cx>
-            <cy>${depth_camera_sub_lens_intri['cx']}</cy>
-            <s>${depth_camera_sub_lens_intri['s']}</s>
-          </intrinsics>
-        </lens>
         <image>
           <width>${depth_camera_sub_image['width']}</width>
