Commit message: feat: add feature to enable args config from ros2 launch
New feature: Enable ROS args config from launch command to set parameters,
such as world model, namespace and initial pose of robot, etc.

Signed-off-by: weijshen <weijshen@qti.qualcomm.com>

File: qrb_ros_sim_gazebo/urdf/gazebo_qrb_mobile_manipulator_robot.urdf.xacro (robot description, xacro)
@@ -3,8 +3,5 @@
 SPDX-License-Identifier: BSD-3-Clause-Clear -->
 <robot xmlns:xacro="http://www.ros.org/wiki/xacro" name="$(arg robot_name)">
-  <xacro:arg name="robot_base_ns" default=""/>
-  <xacro:property name="robot_base_ns_slash" value="${'$(arg robot_base_ns)/' if '$(arg robot_base_ns)' != '' else ''}" />
-  <xacro:arg name="arm_ns" default=""/>
-  <xacro:property name="arm_ns_slash" value="${'$(arg arm_ns)/' if '$(arg arm_ns)' != '' else ''}" />
+  <xacro:arg name="topic_ns" default=""/>
   <!-- Robot base -->
   <xacro:include filename="$(find qrb_ros_sim_description)/urdf/qrb_robot_base/qrb_robot_base.urdf" />
@@ -12,36 +9,40 @@
   <xacro:include filename="$(find qrb_ros_sim_description)/urdf/rml_63_gripper_arm/gripper.urdf" />
   <xacro:include filename="$(find qrb_ros_sim_description)/urdf/orbbec_cameras/gemini335_336.urdf.xacro" />
-  <xacro:qrb_robot_base ns="$(arg robot_base_ns)"/>
-  <xacro:rml_63 ns="$(arg arm_ns)"/>
-  <xacro:rml_gripper ns="$(arg arm_ns)"/>
-  <xacro:gemini_335_336 ns="$(arg arm_ns)"/>
+  <xacro:qrb_robot_base ns=""/>
+  <xacro:rml_63 ns=""/>
+  <xacro:rml_gripper ns=""/>
+  <xacro:gemini_335_336 ns=""/>
   <!-- Gazebo Sensors -->
   <!-- Laser -->
   <xacro:arg name="enable_laser" default="false"/>
-  <xacro:if value="$(arg enable_laser)" >
+  <xacro:arg name="laser_config" default=""/>
+  <xacro:if value="${'$(arg enable_laser)' if '$(arg laser_config)' != '' else 'false'}">
     <xacro:include filename="$(find qrb_ros_sim_gazebo)/urdf/xacro/gazebo_lidar.xacro" />
-    <xacro:gazebo_lidar ns="$(arg robot_base_ns)" reference_link="${robot_base_ns_slash}laser"
-      laser_params_yaml_path="$(find qrb_ros_sim_gazebo)/config/params/qrb_robot_base_laser_params.yaml"/>
+    <xacro:gazebo_lidar ns="" reference_link="laser"
+      laser_params_yaml_path="$(arg laser_config)"/>
   </xacro:if>
   <!-- IMU -->
   <xacro:arg name="enable_imu" default="false"/>
-  <xacro:if value="$(arg enable_imu)" >
+  <xacro:arg name="imu_config" default=""/>
+  <xacro:if value="${'$(arg enable_imu)' if '$(arg imu_config)' != '' else 'false'}">
     <xacro:include filename="$(find qrb_ros_sim_gazebo)/urdf/xacro/gazebo_imu.xacro" />
-    <xacro:gazebo_imu ns="$(arg robot_base_ns)" reference_link="${robot_base_ns_slash}base_imu_link"
-      imu_params_yaml_path="$(find qrb_ros_sim_gazebo)/config/params/imu_params.yaml"/>
+    <xacro:gazebo_imu ns="" reference_link="base_imu_link"
+      imu_params_yaml_path="$(arg imu_config)"/>
   </xacro:if>
   <!-- Arm RGB camera -->
   <xacro:arg name="enable_rgb_camera" default="false"/>
-  <xacro:if value="$(arg enable_rgb_camera)" >
+  <xacro:arg name="rgb_camera_config" default=""/>
+  <xacro:if value="${'$(arg enable_rgb_camera)' if '$(arg rgb_camera_config)' != '' else 'false'}">
     <xacro:include filename="$(find qrb_ros_sim_gazebo)/urdf/xacro/gazebo_rgb_camera.xacro" />
-    <xacro:gazebo_camera ns="$(arg arm_ns)" reference_link="${arm_ns_slash}camera_color_frame"
-      camera_params_yaml_path="$(find qrb_ros_sim_gazebo)/config/params/rgb_camera_params.yaml"/>
+    <xacro:gazebo_camera ns="" reference_link="camera_color_frame"
+      camera_params_yaml_path="$(arg rgb_camera_config)"/>
   </xacro:if>
   <!-- Arm Depth camera -->
   <xacro:arg name="enable_depth_camera" default="false"/>
-  <xacro:if value="$(arg enable_depth_camera)" >
+  <xacro:arg name="depth_camera_config" default=""/>
+  <xacro:if value="${'$(arg enable_depth_camera)' if '$(arg depth_camera_config)' != '' else 'false'}">
     <xacro:include filename="$(find qrb_ros_sim_gazebo)/urdf/xacro/gazebo_depth_camera.xacro" />
-    <xacro:gazebo_depth_camera ns="$(arg arm_ns)" reference_link="${arm_ns_slash}camera_depth_frame"
-      depth_camera_params_yaml_path="$(find qrb_ros_sim_gazebo)/config/params/depth_camera_params.yaml"/>
+    <xacro:gazebo_depth_camera ns="" reference_link="camera_depth_frame"
+      depth_camera_params_yaml_path="$(arg depth_camera_config)"/>
   </xacro:if>
   <!-- Gazebo Plugins -->
@@ -51,22 +52,23 @@
   <xacro:property name="odom_update_rate" value="30"/>
   <xacro:include filename="$(find qrb_ros_sim_gazebo)/urdf/xacro/gazebo_qrb_robot_base_diff_drive.xacro" />
-  <xacro:qrb_robot_base_diff_drive ns="$(arg robot_base_ns)" wheel_separation="${wheel_separation}" separation_multiplier="${separation_multiplier}"
+  <xacro:qrb_robot_base_diff_drive ns="" wheel_separation="${wheel_separation}" separation_multiplier="${separation_multiplier}"
       wheel_radius="${wheel_radius}" radius_multiplier="${radius_multiplier}" update_rate="${odom_update_rate}"/>
   <!-- gz-sim-joint-state-publisher-system controller -->
   <xacro:include filename="$(find qrb_ros_sim_gazebo)/urdf/xacro/gazebo_qrb_robot_base_joint_state_pub.xacro" />
-  <xacro:qrb_robot_base_joint_state_pub ns="$(arg robot_base_ns)"/>
-  <joint name="${robot_base_ns_slash}arm_to_base_joint" type="fixed">
+  <xacro:qrb_robot_base_joint_state_pub ns=""/>
+  <joint name="arm_to_base_joint" type="fixed">
     <origin xyz="0 0 ${box_height/2}" rpy="0 0 ${pi}"/>
-    <parent link="${robot_base_ns_slash}base_link"/>
-    <child link="${arm_ns_slash}arm_base_link"/>
+    <parent link="base_link"/>
+    <child link="arm_base_link"/>
   </joint>
-  <joint name="${arm_ns_slash}arm_camera_joint" type="fixed">
+  <joint name="arm_camera_joint" type="fixed">
     <origin xyz="0.080 0 0.015" rpy="3.1415926 -1.570796 0"/>
-    <parent link="${arm_ns_slash}link6"/>
-    <child link="${arm_ns_slash}camera_link"/>
+    <parent link="link6"/>
+    <child link="camera_link"/>
   </joint>
   <!-- ros2_control -->
   <xacro:include filename="$(find qrb_ros_sim_gazebo)/urdf/xacro/rml_63_gripper_ros2_control.xacro" />
-  <xacro:rml_63_gripper_ros2_control arm_ns="$(arg arm_ns)" robot_desc_ns="$(arg robot_base_ns)"
-      initial_positions_yaml_path="$(find qrb_ros_sim_gazebo)/config/params/initial_positions.yaml"/>
+  <xacro:rml_63_gripper_ros2_control ns="" topic_ns="$(arg topic_ns)"
+      initial_positions_yaml_path="$(find qrb_ros_sim_gazebo)/config/params/initial_positions.yaml"
+      ros2_controllers_yaml_path="$(find qrb_ros_sim_gazebo)/config/params/rml_63_ros2_controllers.yaml"/>
 </robot>

File: qrb_ros_sim_gazebo/urdf/gazebo_qrb_robot_base.urdf.xacro (robot description, xacro)
@@ -3,23 +3,23 @@
 SPDX-License-Identifier: BSD-3-Clause-Clear -->
 <robot xmlns:xacro="http://www.ros.org/wiki/xacro" name="$(arg robot_name)">
-  <xacro:arg name="robot_base_ns" default=""/>
-  <xacro:property name="robot_base_ns_slash" value="${'$(arg robot_base_ns)/' if '$(arg robot_base_ns)' != '' else ''}" />
   <!-- Robot base -->
   <xacro:include filename="$(find qrb_ros_sim_description)/urdf/qrb_robot_base/qrb_robot_base.urdf" />
-  <xacro:qrb_robot_base ns="$(arg robot_base_ns)"/>
+  <xacro:qrb_robot_base ns=""/>
   <!-- Gazebo Sensors -->
   <!-- Laser -->
   <xacro:arg name="enable_laser" default="false"/>
-  <xacro:if value="$(arg enable_laser)" >
+  <xacro:arg name="laser_config" default=""/>
+  <xacro:if value="${'$(arg enable_laser)' if '$(arg laser_config)' != '' else 'false'}">
     <xacro:include filename="$(find qrb_ros_sim_gazebo)/urdf/xacro/gazebo_lidar.xacro" />
-    <xacro:gazebo_lidar ns="$(arg robot_base_ns)" reference_link="${robot_base_ns_slash}laser"
-      laser_params_yaml_path="$(find qrb_ros_sim_gazebo)/config/params/qrb_robot_base_laser_params.yaml"/>
+    <xacro:gazebo_lidar ns="" reference_link="laser"
+      laser_params_yaml_path="$(arg laser_config)"/>
   </xacro:if>
   <!-- IMU -->
   <xacro:arg name="enable_imu" default="false"/>
-  <xacro:if value="$(arg enable_imu)" >
+  <xacro:arg name="imu_config" default=""/>
+  <xacro:if value="${'$(arg enable_imu)' if '$(arg imu_config)' != '' else 'false'}">
     <xacro:include filename="$(find qrb_ros_sim_gazebo)/urdf/xacro/gazebo_imu.xacro" />
-    <xacro:gazebo_imu ns="$(arg robot_base_ns)" reference_link="${robot_base_ns_slash}base_imu_link"
-      imu_params_yaml_path="$(find qrb_ros_sim_gazebo)/config/params/imu_params.yaml"/>
+    <xacro:gazebo_imu ns="" reference_link="base_imu_link"
+      imu_params_yaml_path="$(arg imu_config)"/>
   </xacro:if>
   <!-- Gazebo Plugins -->
@@ -29,8 +29,8 @@
   <xacro:property name="odom_update_rate" value="50"/>
   <xacro:include filename="$(find qrb_ros_sim_gazebo)/urdf/xacro/gazebo_qrb_robot_base_diff_drive.xacro" />
-  <xacro:qrb_robot_base_diff_drive ns="$(arg robot_base_ns)" wheel_separation="${wheel_separation}" separation_multiplier="${separation_multiplier}"
+  <xacro:qrb_robot_base_diff_drive ns="" wheel_separation="${wheel_separation}" separation_multiplier="${separation_multiplier}"
       wheel_radius="${wheel_radius}" radius_multiplier="${radius_multiplier}" update_rate="${odom_update_rate}"/>
   <!-- gz-sim-joint-state-publisher-system controller -->
   <xacro:include filename="$(find qrb_ros_sim_gazebo)/urdf/xacro/gazebo_qrb_robot_base_joint_state_pub.xacro" />
-  <xacro:qrb_robot_base_joint_state_pub ns="$(arg robot_base_ns)"/>
+  <xacro:qrb_robot_base_joint_state_pub ns=""/>
 </robot>

File: qrb_ros_sim_gazebo/urdf/gazebo_qrb_robot_base_mini.urdf.xacro (robot description, xacro)
@@ -3,37 +3,39 @@
 SPDX-License-Identifier: BSD-3-Clause-Clear -->
 <robot xmlns:xacro="http://www.ros.org/wiki/xacro" name="$(arg robot_name)">
-  <xacro:arg name="robot_base_ns" default=""/>
-  <xacro:property name="robot_base_ns_slash" value="${'$(arg robot_base_ns)/' if '$(arg robot_base_ns)' != '' else ''}" />
   <!-- Robot base -->
   <xacro:include filename="$(find qrb_ros_sim_description)/urdf/qrb_robot_base/qrb_robot_base_mini.urdf" />
-  <xacro:qrb_robot_base_mini ns="$(arg robot_base_ns)"/>
+  <xacro:qrb_robot_base_mini ns=""/>
   <!-- Gazebo Sensors -->
   <!-- Laser -->
   <xacro:arg name="enable_laser" default="false"/>
-  <xacro:if value="$(arg enable_laser)" >
+  <xacro:arg name="laser_config" default=""/>
+  <xacro:if value="${'$(arg enable_laser)' if '$(arg laser_config)' != '' else 'false'}">
     <xacro:include filename="$(find qrb_ros_sim_gazebo)/urdf/xacro/gazebo_lidar.xacro" />
-    <xacro:gazebo_lidar ns="$(arg robot_base_ns)" reference_link="${robot_base_ns_slash}laser"
-      laser_params_yaml_path="$(find qrb_ros_sim_gazebo)/config/params/qrb_robot_base_mini_laser_params.yaml"/>
+    <xacro:gazebo_lidar ns="" reference_link="laser"
+      laser_params_yaml_path="$(arg laser_config)"/>
   </xacro:if>
   <!-- IMU -->
   <xacro:arg name="enable_imu" default="false"/>
-  <xacro:if value="$(arg enable_imu)" >
+  <xacro:arg name="imu_config" default=""/>
+  <xacro:if value="${'$(arg enable_imu)' if '$(arg imu_config)' != '' else 'false'}">
     <xacro:include filename="$(find qrb_ros_sim_gazebo)/urdf/xacro/gazebo_imu.xacro" />
-    <xacro:gazebo_imu ns="$(arg robot_base_ns)" reference_link="${robot_base_ns_slash}base_imu_link"
-      imu_params_yaml_path="$(find qrb_ros_sim_gazebo)/config/params/imu_params.yaml"/>
+    <xacro:gazebo_imu ns="" reference_link="base_imu_link"
+      imu_params_yaml_path="$(arg imu_config)"/>
   </xacro:if>
   <!-- RGB camera -->
   <xacro:arg name="enable_rgb_camera" default="false"/>
-  <xacro:if value="$(arg enable_rgb_camera)" >
+  <xacro:arg name="rgb_camera_config" default=""/>
+  <xacro:if value="${'$(arg enable_rgb_camera)' if '$(arg rgb_camera_config)' != '' else 'false'}">
     <xacro:include filename="$(find qrb_ros_sim_gazebo)/urdf/xacro/gazebo_rgb_camera.xacro" />
-    <xacro:gazebo_camera ns="$(arg robot_base_ns)" reference_link="${robot_base_ns_slash}base_camera_color_frame"
-      camera_params_yaml_path="$(find qrb_ros_sim_gazebo)/config/params/rgb_camera_params.yaml"/>
+    <xacro:gazebo_camera ns="" reference_link="base_camera_color_frame"
+      camera_params_yaml_path="$(arg rgb_camera_config)"/>
   </xacro:if>
   <!-- Depth camera -->
   <xacro:arg name="enable_depth_camera" default="false"/>
-  <xacro:if value="$(arg enable_depth_camera)" >
+  <xacro:arg name="depth_camera_config" default=""/>
+  <xacro:if value="${'$(arg enable_depth_camera)' if '$(arg depth_camera_config)' != '' else 'false'}">
     <xacro:include filename="$(find qrb_ros_sim_gazebo)/urdf/xacro/gazebo_depth_camera.xacro" />
-    <xacro:gazebo_depth_camera ns="$(arg robot_base_ns)" reference_link="${robot_base_ns_slash}base_camera_depth_frame"
-      depth_camera_params_yaml_path="$(find qrb_ros_sim_gazebo)/config/params/depth_camera_params.yaml"/>
+    <xacro:gazebo_depth_camera ns="" reference_link="base_camera_depth_frame"
+      depth_camera_params_yaml_path="$(arg depth_camera_config)"/>
   </xacro:if>
   <!-- Gazebo Plugins -->
@@ -43,8 +45,8 @@
   <xacro:property name="odom_update_rate" value="50"/>
   <xacro:include filename="$(find qrb_ros_sim_gazebo)/urdf/xacro/gazebo_qrb_robot_base_diff_drive.xacro" />
-  <xacro:qrb_robot_base_diff_drive ns="$(arg robot_base_ns)" wheel_separation="${wheel_separation}" separation_multiplier="${separation_multiplier}"
+  <xacro:qrb_robot_base_diff_drive ns="" wheel_separation="${wheel_separation}" separation_multiplier="${separation_multiplier}"
       wheel_radius="${wheel_radius}" radius_multiplier="${radius_multiplier}" update_rate="${odom_update_rate}"/>
   <!-- gz-sim-joint-state-publisher-system controller -->
   <xacro:include filename="$(find qrb_ros_sim_gazebo)/urdf/xacro/gazebo_qrb_robot_base_joint_state_pub.xacro" />
-  <xacro:qrb_robot_base_joint_state_pub ns="$(arg robot_base_ns)"/>
+  <xacro:qrb_robot_base_joint_state_pub ns=""/>
 </robot>

File: qrb_ros_sim_gazebo/urdf/gazebo_rml_63_gripper.urdf.xacro (robot description, xacro)
@@ -3,40 +3,42 @@
 SPDX-License-Identifier: BSD-3-Clause-Clear -->
 <robot xmlns:xacro="http://www.ros.org/wiki/xacro" name="$(arg robot_name)">
-  <xacro:arg name="arm_ns" default=""/>
-  <xacro:property name="arm_ns_slash" value="${'$(arg arm_ns)/' if '$(arg arm_ns)' != '' else ''}" />
+  <xacro:arg name="topic_ns" default=""/>
   <!-- Import description urdf file -->
   <xacro:include filename="$(find qrb_ros_sim_description)/urdf/rml_63_gripper_arm/rml_63.urdf" />
   <xacro:include filename="$(find qrb_ros_sim_description)/urdf/rml_63_gripper_arm/gripper.urdf" />
   <xacro:include filename="$(find qrb_ros_sim_description)/urdf/orbbec_cameras/gemini335_336.urdf.xacro" />
-  <xacro:rml_63 ns="$(arg arm_ns)"/>
-  <xacro:rml_gripper ns="$(arg arm_ns)"/>
-  <xacro:gemini_335_336 ns="$(arg arm_ns)"/>
-  <!-- RGB camera -->
+  <xacro:rml_63 ns=""/>
+  <xacro:rml_gripper ns=""/>
+  <xacro:gemini_335_336 ns=""/>
+  <!-- Arm RGB camera -->
   <xacro:arg name="enable_rgb_camera" default="false"/>
-  <xacro:if value="$(arg enable_rgb_camera)" >
+  <xacro:arg name="rgb_camera_config" default=""/>
+  <xacro:if value="${'$(arg enable_rgb_camera)' if '$(arg rgb_camera_config)' != '' else 'false'}">
     <xacro:include filename="$(find qrb_ros_sim_gazebo)/urdf/xacro/gazebo_rgb_camera.xacro" />
-    <xacro:gazebo_camera ns="$(arg arm_ns)" reference_link="${arm_ns_slash}camera_color_frame"
-      camera_params_yaml_path="$(find qrb_ros_sim_gazebo)/config/params/rgb_camera_params.yaml"/>
+    <xacro:gazebo_camera ns="" reference_link="camera_color_frame"
+      camera_params_yaml_path="$(arg rgb_camera_config)"/>
   </xacro:if>
-  <!-- Depth camera -->
+  <!-- Arm Depth camera -->
   <xacro:arg name="enable_depth_camera" default="false"/>
-  <xacro:if value="$(arg enable_depth_camera)" >
+  <xacro:arg name="depth_camera_config" default=""/>
+  <xacro:if value="${'$(arg enable_depth_camera)' if '$(arg depth_camera_config)' != '' else 'false'}">
     <xacro:include filename="$(find qrb_ros_sim_gazebo)/urdf/xacro/gazebo_depth_camera.xacro" />
-    <xacro:gazebo_depth_camera ns="$(arg arm_ns)" reference_link="${arm_ns_slash}camera_depth_frame"
-      depth_camera_params_yaml_path="$(find qrb_ros_sim_gazebo)/config/params/depth_camera_params.yaml"/>
+    <xacro:gazebo_depth_camera ns="" reference_link="camera_depth_frame"
+      depth_camera_params_yaml_path="$(arg depth_camera_config)"/>
   </xacro:if>
-  <joint name="${arm_ns_slash}arm_camera_joint" type="fixed">
+  <joint name="arm_camera_joint" type="fixed">
     <origin xyz="0.080 0 0.015" rpy="3.1415926 -1.570796 0"/>
-    <parent link="${arm_ns_slash}link6"/>
-    <child link="${arm_ns_slash}camera_link"/>
+    <parent link="link6"/>
+    <child link="camera_link"/>
   </joint>
   <link name="world"/>
-  <joint name="${arm_ns_slash}arm_virtual_joint" type="fixed">
+  <joint name="arm_virtual_joint" type="fixed">
     <parent link="world"/>
-    <child link="${arm_ns_slash}arm_base_link"/>
+    <child link="arm_base_link"/>
   </joint>
   <!-- ros2_control -->
   <xacro:include filename="$(find qrb_ros_sim_gazebo)/urdf/xacro/rml_63_gripper_ros2_control.xacro" />
-  <xacro:rml_63_gripper_ros2_control arm_ns="$(arg arm_ns)" robot_desc_ns="$(arg arm_ns)"
-      initial_positions_yaml_path="$(find qrb_ros_sim_gazebo)/config/params/initial_positions.yaml"/>
+  <xacro:rml_63_gripper_ros2_control ns="" topic_ns="$(arg topic_ns)"
+      initial_positions_yaml_path="$(find qrb_ros_sim_gazebo)/config/params/initial_positions.yaml"
+      ros2_controllers_yaml_path="$(find qrb_ros_sim_gazebo)/config/params/rml_63_ros2_controllers.yaml"/>
 </robot>

File: qrb_ros_sim_gazebo/urdf/xacro/gazebo_qrb_robot_base_joint_state_pub.xacro (robot description, xacro)
@@ -5,5 +5,5 @@
     <gazebo>
       <plugin filename="gz-sim-joint-state-publisher-system" name="gz::sim::systems::JointStatePublisher">
-        <topic>${namespace}joint_states</topic>
+        <topic>joint_states</topic>
         <joint_name>${namespace}wheel_right_joint</joint_name>
         <joint_name>${namespace}wheel_left_joint</joint_name>

File: qrb_ros_sim_gazebo/urdf/xacro/rml_63_gripper_ros2_control.xacro (robot description, xacro)
@@ -1,6 +1,6 @@
 <?xml version="1.0"?>
 <robot xmlns:xacro="http://www.ros.org/wiki/xacro">
-  <xacro:macro name="rml_63_gripper_ros2_control" params="arm_ns:='' robot_desc_ns:='' initial_positions_yaml_path">
-    <xacro:property name="namespace" value="${arm_ns + '/' if arm_ns != '' else ''}" />
+  <xacro:macro name="rml_63_gripper_ros2_control" params="ns:='' topic_ns:='' initial_positions_yaml_path ros2_controllers_yaml_path">
+    <xacro:property name="namespace" value="${ns + '/' if ns != '' else ''}" />
     <xacro:property name="initial_positions" value="${xacro.load_yaml(initial_positions_yaml_path)['initial_positions']}"/>
     <!-- ros2_control -->
@@ -81,13 +81,10 @@
     </ros2_control>
     <!-- ros2_control plugin -->
-    <xacro:property name="arm_underscore" value="${arm_ns + '_' if arm_ns != '' else ''}" />
-    <xacro:property name="robot_namespace" value="${robot_desc_ns + '/' if robot_desc_ns != '' else ''}" />
     <gazebo>
       <plugin filename="libgz_ros2_control-system.so" name="gz_ros2_control::GazeboSimROS2ControlPlugin">
         <ros>
-          <namespace>${arm_ns}</namespace>
-          <remapping>/${namespace}robot_description:=/${robot_namespace}robot_description</remapping>
+          <namespace>${topic_ns}</namespace>
         </ros>
-        <parameters>$(find qrb_ros_sim_gazebo)/config/params/${arm_underscore}ros2_controllers.yaml</parameters>
+        <parameters>${ros2_controllers_yaml_path}</parameters>
         <robot_param>robot_description</robot_param>
         <robot_param_node>robot_state_publisher</robot_param_node>
